File: PCB/PICAXEfixer/PICAXEfixer.kicad_pcb (KiCad board)
At the start: 2 copper layers, 83.8 x 38.1 mm, 17 parts, among them J1 MotorConn, J2 SerIn, J3 SerSelect, J4 SerOut, J5 Screw_Terminal_01x04, J6 SerSelect, Q1 KN2222A, U1 PICAXEM2

Commit message: pcb laying out
Parts:
- removed C1: 470uF, Capacitor_THT:CP_Radial_D10.0mm_P5.00mm
- removed C2: 100nF, Capacitor_THT:C_Disc_D4.3mm_W1.9mm_P5.00mm
- removed C3: 10uF, Capacitor_THT:CP_Radial_D5.0mm_P2.50mm
- removed D1: BY126, Diode_THT:D_DO-34_SOD68_P12.70mm_Horizontal
- removed J4: SerOut, Connector_Pin:Pin_D1.0mm_L10.0mm
- removed J5: Screw_Terminal_01x04, TerminalBlock:TerminalBlock_Altech_AK300-4_P5.00mm
- removed J6: SerSelect, Connector_Pin:Pin_D1.0mm_L10.0mm
- removed R4: 1k, Resistor_THT:R_Axial_DIN0414_L11.9mm_D4.5mm_P20.32mm_Horizontal
- removed R5: 18, Resistor_THT:R_Axial_DIN0414_L11.9mm_D4.5mm_P20.32mm_Horizontal
- J1: value MotorConn -> Conn_01x03; footprint Connector_PinHeader_2.54mm:PinHeader_1x04_P2.54mm_Vertical -> Connector_PinHeader_2.54mm:PinHeader_1x03_P2.54mm_Vertical
- J2: value SerIn -> Conn_01x02; footprint Connector_Pin:Pin_D1.0mm_L10.0mm -> Connector_BarrelJack:BarrelJack_Wuerth_6941xx301002
- J3: value SerSelect -> Conn_01x04; footprint Connector_Pin:Pin_D1.0mm_L10.0mm -> Connector_PinHeader_2.54mm:PinHeader_1x04_P2.54mm_Vertical
- Q1: value KN2222A -> 2N7000
- R1: value 1k -> 10k; footprint Resistor_THT:R_Axial_DIN0414_L11.9mm_D4.5mm_P20.32mm_Horizontal -> Resistor_THT:R_Axial_DIN0411_L9.9mm_D3.6mm_P15.24mm_Horizontal
- R2: footprint Resistor_THT:R_Axial_DIN0414_L11.9mm_D4.5mm_P20.32mm_Horizontal -> Resistor_THT:R_Axial_DIN0411_L9.9mm_D3.6mm_P15.24mm_Horizontal
- R3: value 22k -> 10k; footprint Resistor_THT:R_Axial_DIN0414_L11.9mm_D4.5mm_P20.32mm_Horizontal -> Resistor_THT:R_Axial_DIN0411_L9.9mm_D3.6mm_P15.24mm_Horizontal
- U1: footprint Package_DIP:DIP-8_W10.16mm -> Package_DIP:DIP-8_W7.62mm
- moved R2 56.4 mm to (83.8, 19.1), turned to 0 degrees
- moved J3 44.2 mm to (74.9, 31.8)
- moved Q1 42.7 mm to (115.6, 44.5), turned to 270 degrees
- moved J2 30.2 mm to (139.7, 34.3), turned to 90 degrees
- moved R1 28.1 mm to (124.5, 50.8), turned to 0 degrees
- moved U1 24.2 mm to (87.6, 31.8)
- moved J1 17.8 mm to (74.9, 45.7)
- moved R3 13.7 mm to (101.6, 40.6)
Connections:
- J1 pad 3: Net-(C1-Pad2) -> Net-(J1-Pad3)
- J2 pad 1: Net-(J2-Pad1) -> GNDD
- J3 pad 1: Net-(J3-Pad1) -> +5P
- Q1 pad 2: Net-(Q1-Pad2) -> Net-(J1-Pad2)
- Q1 pad 3: Net-(C1-Pad2) -> Net-(Q1-Pad3)
- R1 pad 1: Net-(R1-Pad1) -> Net-(Q1-Pad3)
- R1 pad 2: Net-(J1-Pad2) -> +5P
- R2 pad 1: Net-(J2-Pad1) -> Net-(R2-Pad1)
- R3 pad 2: Net-(J2-Pad1) -> Net-(Q1-Pad3)
- U1 pad 2: Net-(R3-Pad1) -> Net-(R2-Pad1)
- U1 pad 3: Net-(J3-Pad1) -> (no net)
- U1 pad 4: Net-(R1-Pad1) -> (no net)
- U1 pad 5: Net-(U1-Pad5) -> (no net)
- U1 pad 6: Net-(R4-Pad1) -> Net-(R3-Pad1)
- U1 pad 7: Net-(J4-Pad1) -> Net-(J3-Pad3)
Routing:
- net GNDD: track 198.3 -> 0.00 mm
- net +5P: track 71.0 -> 0.00 mm
- net +5C: track 48.3 -> 0.00 mm
- net Net-(R4-Pad1): track 45.7 -> 0.00 mm
- net Net-(J1-Pad2): track 43.2 -> 0.00 mm
- net Net-(J2-Pad1): track 35.6 -> 0.00 mm
- net Net-(C1-Pad1): track 35.6 -> 0.00 mm
- net Net-(Q1-Pad2): track 29.5 -> 0.00 mm
- net Net-(C1-Pad2): track 27.8 -> 0.00 mm
- net Net-(R1-Pad1): track 22.9 -> 0.00 mm
- net Net-(J3-Pad1): track 17.8 -> 0.00 mm
- net Net-(J4-Pad1): track 15.2 -> 0.00 mm
- net Net-(R3-Pad1): track 12.7 -> 0.00 mm

Commit message: PCB laid out
Parts:
- added C1: 100uF, Capacitor_THT:CP_Radial_D10.0mm_P5.00mm, F.Cu at (76.2, 26.7)
- added C2: 100nF, Capacitor_THT:C_Disc_D4.3mm_W1.9mm_P5.00mm, F.Cu at (88.9, 26.7)
- added R4: 10k, Resistor_THT:R_Axial_DIN0309_L9.0mm_D3.2mm_P15.24mm_Horizontal, F.Cu at (78.7, 43.2)
- R1, R2, R3: footprint Resistor_THT:R_Axial_DIN0411_L9.9mm_D3.6mm_P15.24mm_Horizontal -> Resistor_THT:R_Axial_DIN0309_L9.0mm_D3.2mm_P15.24mm_Horizontal
- moved J2 40.1 mm to (100.3, 26.7)
- moved Q1 29.9 mm to (86.4, 50.8), turned to 90 degrees
- moved R1 20.4 mm to (104.1, 52.1), turned to 90 degrees
- moved R2 20.3 mm to (83.8, 39.4), turned to 90 degrees
- moved R3 4.58 mm to (99.1, 36.8)
Connections:
- U1 pad 7: Net-(J3-Pad3) -> Net-(R4-Pad2)
Routing:
- net GNDD: track 0.00 -> 97.6 mm
- net +5P: track 0.00 -> 87.1 mm
- net Net-(J1-Pad3): track 0.00 -> 29.2 mm
- net Net-(J1-Pad2): track 0.00 -> 22.8 mm
- net Net-(Q1-Pad3): track 0.00 -> 21.7 mm
- net Net-(R4-Pad2): track 0.00 -> 12.7 mm
- net Net-(J3-Pad3): track 0.00 -> 10.2 mm
- net Net-(R2-Pad1): track 0.00 -> 8.89 mm
- net Net-(R3-Pad1): track 0.00 -> 3.81 mm
Other:
- board size 83.8 x 38.1 mm -> 48.3 x 38.1 mm

Commit message: final
Parts:
- C1: footprint Capacitor_THT:CP_Radial_D10.0mm_P5.00mm -> Capacitor_THT:CP_Radial_D10.0mm_P7.50mm
- C2: footprint Capacitor_THT:C_Disc_D4.3mm_W1.9mm_P5.00mm -> Capacitor_THT:C_Disc_D7.5mm_W5.0mm_P10.00mm
- moved J2 3.81 mm to (100.3, 30.5)
- moved C2 1.27 mm to (87.6, 26.7)
- moved C1 1.27 mm to (76.2, 27.9)
Connections:
- J2 pad 1: GNDD -> +5P
- J2 pad 2: +5P -> GNDD
Routing:
- net GNDD: track 97.6 -> 120.8 mm
- net +5P: track 87.1 -> 90.2 mm

Commit message: Circuit built & testing, functions erratically :/
Parts:
- added J4: Jumper, Connector_PinHeader_2.54mm:PinHeader_1x02_P2.54mm_Vertical, F.Cu at (108.0, 45.7)
- J1: value Conn_01x03 -> From PC
- J2: value Conn_01x02 -> Power
- J3: value Conn_01x04 -> To PICAXE
- moved Q1 1.27 mm to (86.4, 52.1)
Connections:
- U1 pad 4: (no net) -> Net-(J4-Pad1)
Routing:
- net Net-(J4-Pad1): track 0.00 -> 30.7 mm
- net GNDD: track 120.8 -> 132.2 mm
- net Net-(Q1-Pad3): track 21.7 -> 20.3 mm

Commit message: finally works
Parts:
- added R5: 10k, Resistor_THT:R_Axial_DIN0309_L9.0mm_D3.2mm_P15.24mm_Horizontal, F.Cu at (110.5, 38.1)
- added R6: 10k, Resistor_THT:R_Axial_DIN0309_L9.0mm_D3.2mm_P15.24mm_Horizontal, F.Cu at (81.3, 34.3)
- J1: footprint Connector_PinHeader_2.54mm:PinHeader_1x03_P2.54mm_Vertical -> Connector_PinHeader_2.54mm:PinHeader_1x04_P2.54mm_Vertical
- moved J4 6.35 mm to (114.3, 45.7)
- moved J1 2.54 mm to (74.9, 43.2)
- moved R4 1.27 mm to (77.5, 43.2)
Connections:
- net Net-(J1-Pad2) renamed /TxD
- net Net-(J1-Pad3) renamed /RxD
- U1 pad 3: (no net) -> Net-(R6-Pad1)
Routing:
- net Net-(R6-Pad1): track 0.00 -> 18.2 mm
- net Net-(J4-Pad1): track 30.7 -> 42.2 mm
- net +5P: track 90.2 -> 97.8 mm
- net /CTS: track 0.00 -> 7.62 mm
- net /RxD: track 29.2 -> 22.0 mm
- net GNDD: track 132.2 -> 138.5 mm
- net /TxD: track 22.7 -> 25.4 mm
- net Net-(J3-Pad3): track 10.2 -> 8.89 mm
